File: hardware/wifi-extension.kicad_pcb (KiCad board)
At the start: 2 copper layers, 40 x 40 mm, 35 parts, among them J1 STACK-UP-HIGH, J2 STACK-DOWN, J3 STACK-UP-HIGH, J4 STACK-DOWN, P1 CONN_1, P2 CONN_1, P3 CONN_1, U1 M24C64, U2 ESP8266_WROOM02, U3 DRILL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

Commit message: Add 3d information (final)
Parts:
- C1, C2: footprint kicad-libraries:0603E -> kicad-libraries:C0603E
- C3: footprint kicad-libraries:0805E -> kicad-libraries:C0805E
- R1, R2, R3, R4: footprint kicad-libraries:0603E -> kicad-libraries:R0603E
Connections:
- FILTER1 pad 11: (no net) -> Net-(FILTER1-Pad11)
- FILTER1 pad 13: (no net) -> Net-(FILTER1-Pad13)
- FILTER1 pad 15: (no net) -> Net-(FILTER1-Pad15)
- FILTER1 pad 2: (no net) -> Net-(FILTER1-Pad2)
- FILTER1 pad 4: (no net) -> Net-(FILTER1-Pad4)
- FILTER1 pad 6: (no net) -> Net-(FILTER1-Pad6)
- FILTER1 pad 8: (no net) -> Net-(FILTER1-Pad8)
- FILTER1 pad 9: (no net) -> Net-(FILTER1-Pad9)
- J1 pad 25: (no net) -> Net-(J1-Pad25)
- J1 pad 27: (no net) -> Net-(J1-Pad27)
- J1 pad 29: (no net) -> Net-(J1-Pad29)
- RP1 pad 2: (no net) -> Net-(RP1-Pad2)
- RP1 pad 3: (no net) -> Net-(RP1-Pad3)
- RP1 pad 6: (no net) -> Net-(RP1-Pad6)
- RP1 pad 7: (no net) -> Net-(RP1-Pad7)
- RP2 pad 2: (no net) -> Net-(RP2-Pad2)
- RP2 pad 3: (no net) -> Net-(RP2-Pad3)
- RP2 pad 6: (no net) -> Net-(RP2-Pad6)
- RP2 pad 7: (no net) -> Net-(RP2-Pad7)
- U1 pad 7: (no net) -> Net-(U1-Pad7)
- U2 pad 16: (no net) -> Net-(U2-Pad16)
- U2 pad 17: (no net) -> Net-(U2-Pad17)
- U2 pad 5: (no net) -> Net-(U2-Pad5)
